Commit message: spwaned in gazebo with no error and one warning

File: advr_mob_plt_description/urdf/main.urdf (robot description, URDF)
Before this commit: robot MAIN, 5 links, 4 joints
Links:
- added link footprint
Joints:
- removed joint CHASSIS_SUB--WHEEL_SUB
- removed joint CHASSIS_SUB--WHEEL_SUB-1
- removed joint CHASSIS_SUB--WHEEL_SUB-2
- removed joint CHASSIS_SUB--WHEEL_SUB-3
- added joint CHASSIS_SUB_WHEEL_SUB: type continuous, parent CHASSIS_SUB, child WHEEL_SUB, origin xyz=10.9855 -3.175 0.635 rpy=3.14159265359 -0.773676769918 0, axis 0.0 -1.0 0.0
- added joint CHASSIS_SUB_WHEEL_SUB_1: type continuous, parent CHASSIS_SUB, child WHEEL_SUB-1, origin xyz=1.4605 3.175 0.635 rpy=0 0.731481857872 3.14159265359, axis 0.0 1.0 0.0
- added joint CHASSIS_SUB_WHEEL_SUB_2: type continuous, parent CHASSIS_SUB, child WHEEL_SUB-2, origin xyz=10.9855 -3.175 0.635 rpy=0 0.157649211716 0, axis 0.0 1.0 0.0
- added joint CHASSIS_SUB_WHEEL_SUB_3: type continuous, parent CHASSIS_SUB, child WHEEL_SUB-3, origin xyz=1.4605 3.175 0.635 rpy=0 -1.30226592388 0, axis 0.0 -1.0 0.0
- added joint base_joint: type fixed, parent footprint, child CHASSIS_SUB
